File: powerglove_pcb/powerglove_pcb.sch (KiCad schematic (older format))
At the start: 17 parts, among them J1 Conn_01x07, J2 Conn_01x07, J3 Conn_01x02, J4 Conn_01x05, J5 Conn_01x03, J6 Conn_01x03, Q1 BSS123, Q2 BSS123, U1 DRV2605

Commit message: updated schematic with assigned footprints, ported into layout
Parts:
- added J1: Conn_01x02, Connector_PinHeader_2.54mm:PinHeader_1x02_P2.54mm_Vertical, symbol Connector_Generic:Conn_01x02
- C1, C2: footprint (none) -> Capacitor_SMD:C_0603_1608Metric_Pad1.05x0.95mm_HandSolder
- J2: renamed from J1; value Conn_01x07 -> Conn_01x05; footprint (none) -> Connector_PinHeader_2.54mm:PinHeader_1x05_P2.54mm_Vertical; symbol Connector_Generic:Conn_01x07 -> Connector_Generic:Conn_01x05
- J3: renamed from J2; footprint (none) -> Connector_PinHeader_2.54mm:PinHeader_1x07_P2.54mm_Vertical
- J4: renamed from J3; footprint (none) -> Connector_PinHeader_2.54mm:PinHeader_2x01_P2.54mm_Vertical
- J5: renamed from J4; footprint (none) -> Connector_PinHeader_2.54mm:PinHeader_1x05_P2.54mm_Vertical
- J6: renamed from J5; footprint (none) -> Connector_PinHeader_2.54mm:PinHeader_1x03_P2.54mm_Vertical
- J7: renamed from J6; footprint (none) -> Connector_PinHeader_2.54mm:PinHeader_1x03_P2.54mm_Vertical
- R1, R2, R3, R4, R5, R6: footprint (none) -> Resistor_SMD:R_0603_1608Metric_Pad1.05x0.95mm_HandSolder
- U1: footprint (none) -> Package_SO:VSSOP-10_3x3mm_P0.5mm
Connections:
- net GND: now also J1.2 (Pin_2)
- net VBAT: now also J1.1 (Pin_1); no longer J2.7 (Pin_7)
- no-connect marks 2 -> 1
Other:
- note added: "From Battery (2S Lipo)"
- note added: "To Buckler (header connection)"
- note added: "To Buckler (jumpers)\n"
- moved on the sheet: J3

Commit message: Added ToF sensor header, arrange layout
Parts:
- added J8: Conn_01x07, Connector_PinHeader_2.54mm:PinHeader_1x07_P2.54mm_Vertical, symbol Connector_Generic:Conn_01x07
- U1: symbol powerglove_library:DRV2605 -> powerglove_pcb-rescue:DRV2605-powerglove_library
Connections:
- wire segments 69 -> 75
- no-connect marks 1 -> 4
Other:
- note added: "ToF Sensor"
Changed lines of the file:
@@
 EESchema Schematic File Version 4
+LIBS:powerglove_pcb-cache
 EELAYER 30 0
 EELAYER END
@@
 $EndDescr
 $Comp
-L powerglove_library:DRV2605 U1
+L powerglove_pcb-rescue:DRV2605-powerglove_library U1
 U 1 1 5FA9BF1E
 P 5400 3400
@@
 Text Notes 1950 2250 0    50   ~ 0
 From Battery (2S Lipo)
+$Comp
+L Connector_Generic:Conn_01x07 J8
+U 1 1 5FAEEE70
+P 2450 6150
+F 0 "J8" H 2368 5625 50  0000 C CNN
+F 1 "Conn_01x07" H 2368 5716 50  0000 C CNN
+F 2 "Connector_PinHeader_2.54mm:PinHeader_1x07_P2.54mm_Vertical" H 2450 6150 50  0001 C CNN
+F 3 "~" H 2450 6150 50  0001 C CNN
+	1    2450 6150
+	-1   0    0    1
+$EndComp
+Text Notes 2300 5500 0    50   ~ 0
+ToF Sensor
+Wire Wire Line
+	2650 6150 2900 6150
+Wire Wire Line
+	2650 6250 2900 6250
+Text Label 2900 6250 0    50   ~ 0
+SCL
+Text Label 2900 6150 0    50   ~ 0
+SDA
+Wire Wire Line
+	3150 6050 3150 6100
+Wire Wire Line
+	2650 6050 3150 6050
+$Comp
+L power:GND #PWR024
+U 1 1 5FAF6B54
+P 3150 6100
+F 0 "#PWR024" H 3150 5850 50  0001 C CNN
+F 1 "GND" H 3155 5927 50  0000 C CNN
+F 2 "" H 3150 6100 50  0001 C CNN
+F 3 "" H 3150 6100 50  0001 C CNN
+	1    3150 6100
+	1    0    0    -1
+$EndComp
+$Comp
+L power:+3V3 #PWR023
+U 1 1 5FAF9080
+P 3150 5900
+F 0 "#PWR023" H 3150 5750 50  0001 C CNN
+F 1 "+3V3" H 3165 6073 50  0000 C CNN
+F 2 "" H 3150 5900 50  0001 C CNN
+F 3 "" H 3150 5900 50  0001 C CNN
+	1    3150 5900
+	1    0    0    -1
+$EndComp
+Wire Wire Line
+	3150 5950 3150 5900
+Wire Wire Line
+	2650 5950 3150 5950
+NoConn ~ 2650 6450
+NoConn ~ 2650 6350
+NoConn ~ 2650 5850
 $EndSCHEMATC

Commit message: PCB layout complete
Parts:
- removed J8: Conn_01x07, Connector_PinHeader_2.54mm:PinHeader_1x07_P2.54mm_Vertical, symbol Connector_Generic:Conn_01x07
- removed U1: DRV2605, Package_SO:VSSOP-10_3x3mm_P0.5mm, symbol powerglove_pcb-rescue:DRV2605-powerglove_library
- added J8: Conn_01x04, Connector_PinHeader_2.54mm:PinHeader_1x04_P2.54mm_Vertical, symbol Connector_Generic:Conn_01x04
- added U1: DRV2605, Package_SO:VSSOP-10_3x3mm_P0.5mm, symbol powerglove_library:DRV2605
Connections:
- no-connect marks 4 -> 1
Changed lines of the file:
@@
 $EndDescr
-$Comp
-L powerglove_pcb-rescue:DRV2605-powerglove_library U1
-U 1 1 5FA9BF1E
-P 5400 3400
-F 0 "U1" H 5700 2950 50  0000 C CNN
-F 1 "DRV2605" H 5800 2850 50  0000 C CNN
-F 2 "Package_SO:VSSOP-10_3x3mm_P0.5mm" H 5400 3400 50  0001 C CNN
-F 3 "" H 5400 3400 50  0001 C CNN
-	1    5400 3400
-	1    0    0    -1
-$EndComp
 $Comp
 L Device:C C2
@@
 Text Label 2900 3700 0    50   ~ 0
 INT
+Text Label 2900 3900 0    50   ~ 0
+SERVO1
 Text Label 2900 3800 0    50   ~ 0
-SERVO1
-Text Label 2900 3900 0    50   ~ 0
 SERVO2
 Wire Wire Line
@@
 Text Notes 1950 2250 0    50   ~ 0
 From Battery (2S Lipo)
-$Comp
-L Connector_Generic:Conn_01x07 J8
-U 1 1 5FAEEE70
-P 2450 6150
-F 0 "J8" H 2368 5625 50  0000 C CNN
-F 1 "Conn_01x07" H 2368 5716 50  0000 C CNN
-F 2 "Connector_PinHeader_2.54mm:PinHeader_1x07_P2.54mm_Vertical" H 2450 6150 50  0001 C CNN
-F 3 "~" H 2450 6150 50  0001 C CNN
-	1    2450 6150
-	-1   0    0    1
-$EndComp
 Text Notes 2300 5500 0    50   ~ 0
 ToF Sensor
@@
 Wire Wire Line
 	2650 5950 3150 5950
-NoConn ~ 2650 6450
-NoConn ~ 2650 6350
-NoConn ~ 2650 5850
+$Comp
+L Connector_Generic:Conn_01x04 J8
+U 1 1 5FAF6479
+P 2450 6150
+F 0 "J8" H 2368 5725 50  0000 C CNN
+F 1 "Conn_01x04" H 2368 5816 50  0000 C CNN
+F 2 "Connector_PinHeader_2.54mm:PinHeader_1x04_P2.54mm_Vertical" H 2450 6150 50  0001 C CNN
+F 3 "~" H 2450 6150 50  0001 C CNN
+	1    2450 6150
+	-1   0    0    1
+$EndComp
+$Comp
+L powerglove_library:DRV2605 U1
+U 1 1 5FB13902
+P 5400 3400
+F 0 "U1" H 5750 2950 50  0000 C CNN
+F 1 "DRV2605" H 5850 2850 50  0000 C CNN
+F 2 "Package_SO:VSSOP-10_3x3mm_P0.5mm" H 5400 3400 50  0001 C CNN
+F 3 "https://www.ti.com/lit/ds/symlink/drv2605l.pdf" H 5400 3400 50  0001 C CNN
+	1    5400 3400
+	1    0    0    -1
+$EndComp
 $EndSCHEMATC

Commit message: update PCB layout for simple battery monitoring, clean up silk
Parts:
- added R7, R8, R9: 10k, Resistor_SMD:R_0603_1608Metric_Pad1.05x0.95mm_HandSolder, symbol Device:R
- J2: value Conn_01x05 -> Conn_01x06; footprint Connector_PinHeader_2.54mm:PinHeader_1x05_P2.54mm_Vertical -> Connector_PinHeader_2.54mm:PinHeader_1x06_P2.54mm_Vertical; symbol Connector_Generic:Conn_01x05 -> Connector_Generic:Conn_01x06
Connections:
- net GND: now also R9.2
- net VBAT: now also R7.1
- new net: R7.2, R8.1
- new net monitor: J2.6 (Pin_6), R8.2, R9.1
Other:
- note added: "Divider for Battery Monitoring\n"
- moved on the sheet: J3, J8
Changed lines of the file:
@@
 EESchema Schematic File Version 4
-LIBS:powerglove_pcb-cache
 EELAYER 30 0
 EELAYER END
@@
 PG
 $Comp
-L Connector_Generic:Conn_01x05 J2
+L Connector_Generic:Conn_01x06 J2
 U 1 1 5FB32D8E
 P 2450 3700
 F 0 "J2" H 2368 3175 50  0000 C CNN
-F 1 "Conn_01x05" H 2368 3266 50  0000 C CNN
-F 2 "Connector_PinHeader_2.54mm:PinHeader_1x05_P2.54mm_Vertical" H 2450 3700 50  0001 C CNN
+F 1 "Conn_01x06" H 2368 3266 50  0000 C CNN
+F 2 "Connector_PinHeader_2.54mm:PinHeader_1x06_P2.54mm_Vertical" H 2450 3700 50  0001 C CNN
 F 3 "~" H 2450 3700 50  0001 C CNN
 	1    2450 3700
@@
 Wire Wire Line
 	2650 2700 2900 2700
-Text Notes 1950 4200 0    50   ~ 0
+Text Notes 1950 4400 0    50   ~ 0
 To Buckler (header connection)
 $Comp
 L power:GND #PWR01
 U 1 1 5FB2FC84
-P 2750 5150
-F 0 "#PWR01" H 2750 4900 50  0001 C CNN
-F 1 "GND" H 2755 4977 50  0000 C CNN
-F 2 "" H 2750 5150 50  0001 C CNN
-F 3 "" H 2750 5150 50  0001 C CNN
-	1    2750 5150
-	1    0    0    -1
-$EndComp
-Wire Wire Line
-	2750 5100 2750 5150
-Connection ~ 2750 5100
-Wire Wire Line
-	2650 5100 2750 5100
-Wire Wire Line
-	2750 5000 2750 5100
-Wire Wire Line
-	2650 5000 2750 5000
+P 2750 5350
+F 0 "#PWR01" H 2750 5100 50  0001 C CNN
+F 1 "GND" H 2755 5177 50  0000 C CNN
+F 2 "" H 2750 5350 50  0001 C CNN
+F 3 "" H 2750 5350 50  0001 C CNN
+	1    2750 5350
+	1    0    0    -1
+$EndComp
+Wire Wire Line
+	2750 5300 2750 5350
+Connection ~ 2750 5300
+Wire Wire Line
+	2650 5300 2750 5300
+Wire Wire Line
+	2750 5200 2750 5300
+Wire Wire Line
+	2650 5200 2750 5200
 $Comp
 L power:+3V3 #PWR02
 U 1 1 5FB2C6C7
-P 2850 4500
-F 0 "#PWR02" H 2850 4350 50  0001 C CNN
-F 1 "+3V3" H 2865 4673 50  0000 C CNN
-F 2 "" H 2850 4500 50  0001 C CNN
-F 3 "" H 2850 4500 50  0001 C CNN
-	1    2850 4500
+P 2850 4700
+F 0 "#PWR02" H 2850 4550 50  0001 C CNN
+F 1 "+3V3" H 2865 4873 50  0000 C CNN
+F 2 "" H 2850 4700 50  0001 C CNN
+F 3 "" H 2850 4700 50  0001 C CNN
+	1    2850 4700
 	1    0    0    -1
 $EndComp
@@
 L power:+5V #PWR03
 U 1 1 5FB2C441
-P 2850 4900
-F 0 "#PWR03" H 2850 4750 50  0001 C CNN
-F 1 "+5V" H 2865 5073 50  0000 C CNN
-F 2 "" H 2850 4900 50  0001 C CNN
-F 3 "" H 2850 4900 50  0001 C CNN
-	1    2850 4900
-	1    0    0    -1
-$EndComp
-Wire Wire Line
-	2650 4900 2850 4900
+P 2850 5100
+F 0 "#PWR03" H 2850 4950 50  0001 C CNN
+F 1 "+5V" H 2865 5273 50  0000 C CNN
+F 2 "" H 2850 5100 50  0001 C CNN
+F 3 "" H 2850 5100 50  0001 C CNN
+	1    2850 5100
+	1    0    0    -1
+$EndComp
+Wire Wire Line
+	2650 5100 2850 5100
 $Comp
 L Connector_Generic:Conn_01x07 J3
 U 1 1 5FB2A376
-P 2450 4800
-F 0 "J3" H 2368 4275 50  0000 C CNN
-F 1 "Conn_01x07" H 2368 4366 50  0000 C CNN
-F 2 "Connector_PinHeader_2.54mm:PinHeader_1x07_P2.54mm_Vertical" H 2450 4800 50  0001 C CNN
-F 3 "~" H 2450 4800 50  0001 C CNN
-	1    2450 4800
+P 2450 5000
+F 0 "J3" H 2368 4475 50  0000 C CNN
+F 1 "Conn_01x07" H 2368 4566 50  0000 C CNN
+F 2 "Connector_PinHeader_2.54mm:PinHeader_1x07_P2.54mm_Vertical" H 2450 5000 50  0001 C CNN
+F 3 "~" H 2450 5000 50  0001 C CNN
+	1    2450 5000
 	-1   0    0    1
 $EndComp
-NoConn ~ 2650 4700
-Connection ~ 2750 4600
-Wire Wire Line
-	2750 4800 2750 4600
+NoConn ~ 2650 4900
+Connection ~ 2750 4800
+Wire Wire Line
+	2750 5000 2750 4800
+Wire Wire Line
+	2650 5000 2750 5000
+Wire Wire Line
+	2750 4700 2850 4700
+Connection ~ 2750 4700
+Wire Wire Line
+	2750 4800 2750 4700
 Wire Wire Line
 	2650 4800 2750 4800
 Wire Wire Line
-	2750 4500 2850 4500
-Connection ~ 2750 4500
-Wire Wire Line
-	2750 4600 2750 4500
-Wire Wire Line
-	2650 4600 2750 4600
-Wire Wire Line
-	2650 4500 2750 4500
+	2650 4700 2750 4700
 Text Notes 1950 3100 0    50   ~ 0
 To Buckler (jumpers)\n
 Text Notes 1950 2250 0    50   ~ 0
 From Battery (2S Lipo)
-Text Notes 2300 5500 0    50   ~ 0
+Text Notes 2150 5750 0    50   ~ 0
 ToF Sensor
 Wire Wire Line
-	2650 6150 2900 6150
-Wire Wire Line
 	2650 6250 2900 6250
+Wire Wire Line
+	2650 6350 2900 6350
+Text Label 2900 6350 0    50   ~ 0
+SCL
 Text Label 2900 6250 0    50   ~ 0
-SCL
-Text Label 2900 6150 0    50   ~ 0
 SDA
 Wire Wire Line
-	3150 6050 3150 6100
-Wire Wire Line
-	2650 6050 3150 6050
+	3150 6150 3150 6200
+Wire Wire Line
+	2650 6150 3150 6150
 $Comp
 L power:GND #PWR024
 U 1 1 5FAF6B54
-P 3150 6100
-F 0 "#PWR024" H 3150 5850 50  0001 C CNN
-F 1 "GND" H 3155 5927 50  0000 C CNN
-F 2 "" H 3150 6100 50  0001 C CNN
-F 3 "" H 3150 6100 50  0001 C CNN
-	1    3150 6100
+P 3150 6200
+F 0 "#PWR024" H 3150 5950 50  0001 C CNN
+F 1 "GND" H 3155 6027 50  0000 C CNN
+F 2 "" H 3150 6200 50  0001 C CNN
+F 3 "" H 3150 6200 50  0001 C CNN
+	1    3150 6200
 	1    0    0    -1
 $EndComp
@@
 L power:+3V3 #PWR023
 U 1 1 5FAF9080
-P 3150 5900
-F 0 "#PWR023" H 3150 5750 50  0001 C CNN
-F 1 "+3V3" H 3165 6073 50  0000 C CNN
-F 2 "" H 3150 5900 50  0001 C CNN
-F 3 "" H 3150 5900 50  0001 C CNN
-	1    3150 5900
-	1    0    0    -1
-$EndComp
-Wire Wire Line
-	3150 5950 3150 5900
-Wire Wire Line
-	2650 5950 3150 5950
-$Comp
-L Connector_Generic:Conn_01x04 J8
-U 1 1 5FAF6479
-P 2450 6150
-F 0 "J8" H 2368 5725 50  0000 C CNN
-F 1 "Conn_01x04" H 2368 5816 50  0000 C CNN
-F 2 "Connector_PinHeader_2.54mm:PinHeader_1x04_P2.54mm_Vertical" H 2450 6150 50  0001 C CNN
-F 3 "~" H 2450 6150 50  0001 C CNN
-	1    2450 6150
-	-1   0    0    1
-$EndComp
+P 3150 6000
+F 0 "#PWR023" H 3150 5850 50  0001 C CNN
+F 1 "+3V3" H 3165 6173 50  0000 C CNN
+F 2 "" H 3150 6000 50  0001 C CNN
+F 3 "" H 3150 6000 50  0001 C CNN
+	1    3150 6000
+	1    0    0    -1
+$EndComp
+Wire Wire Line
+	3150 6050 3150 6000
+Wire Wire Line
+	2650 6050 3150 6050
 $Comp
 L powerglove_library:DRV2605 U1
@@
 	1    0    0    -1
 $EndComp
+$Comp
+L Device:R R7
+U 1 1 5FAF0DDB
+P 4300 5200
+F 0 "R7" H 4370 5246 50  0000 L CNN
+F 1 "10k" H 4370 5155 50  0000 L CNN
+F 2 "Resistor_SMD:R_0603_1608Metric_Pad1.05x0.95mm_HandSolder" V 4230 5200 50  0001 C CNN
+F 3 "~" H 4300 5200 50  0001 C CNN
+	1    4300 5200
+	1    0    0    -1
+$EndComp
+$Comp
+L Device:R R8
+U 1 1 5FAF2A87
+P 4300 5600
+F 0 "R8" H 4370 5646 50  0000 L CNN
+F 1 "10k" H 4370 5555 50  0000 L CNN
+F 2 "Resistor_SMD:R_0603_1608Metric_Pad1.05x0.95mm_HandSolder" V 4230 5600 50  0001 C CNN
+F 3 "~" H 4300 5600 50  0001 C CNN
+	1    4300 5600
+	1    0    0    -1
+$EndComp
+$Comp
+L Device:R R9
+U 1 1 5FAF4D96
+P 4300 6050
+F 0 "R9" H 4370 6096 50  0000 L CNN
+F 1 "10k" H 4370 6005 50  0000 L CNN
+F 2 "Resistor_SMD:R_0603_1608Metric_Pad1.05x0.95mm_HandSolder" V 4230 6050 50  0001 C CNN
+F 3 "~" H 4300 6050 50  0001 C CNN
+	1    4300 6050
+	1    0    0    -1
+$EndComp
+Text Label 4300 4950 0    50   ~ 0
+VBAT
+Wire Wire Line
+	4300 4950 4300 5050
+Wire Wire Line
+	4300 5350 4300 5450
+Wire Wire Line
+	4300 5750 4300 5800
+$Comp
+L power:GND #PWR025
+U 1 1 5FB03B96
+P 4300 6200
+F 0 "#PWR025" H 4300 5950 50  0001 C CNN
+F 1 "GND" H 4305 6027 50  0000 C CNN
+F 2 "" H 4300 6200 50  0001 C CNN
+F 3 "" H 4300 6200 50  0001 C CNN
+	1    4300 6200
+	1    0    0    -1
+$EndComp
+Text Label 4650 5800 0    50   ~ 0
+monitor
+Wire Wire Line
+	4650 5800 4300 5800
+Connection ~ 4300 5800
+Wire Wire Line
+	4300 5800 4300 5900
+$Comp
+L Connector_Generic:Conn_01x04 J8
+U 1 1 5FAF6479
+P 2450 6250
+F 0 "J8" H 2368 5825 50  0000 C CNN
+F 1 "Conn_01x04" H 2368 5916 50  0000 C CNN
+F 2 "Connector_PinHeader_2.54mm:PinHeader_1x04_P2.54mm_Vertical" H 2450 6250 50  0001 C CNN
+F 3 "~" H 2450 6250 50  0001 C CNN
+	1    2450 6250
+	-1   0    0    1
+$EndComp
+Text Label 2900 3400 0    50   ~ 0
+monitor
+Wire Wire Line
+	2900 3400 2650 3400
+Text Notes 4150 4750 0    50   ~ 0
+Divider for Battery Monitoring\n
+Wire Notes Line
+	4100 4550 5350 4550
+Wire Notes Line
+	5350 4550 5350 6500
+Wire Notes Line
+	5350 6500 4100 6500
+Wire Notes Line
+	4100 6500 4100 4550
 $EndSCHEMATC
